File: rv_cad/JA972/JA972.kicad_pcb (KiCad board)
At the start: 2 copper layers, 160 x 100 mm, 112 parts, among them J1 Conn_Coaxial, J10 P10, J11 P11, J12 E2, J13 E3, J14 P6, J15 P2, J16 P4, J17 P1, J18 P3, J19 P5, J2 PGM_SWITCH1, J20 P5, J21 P5, J3 PGM_SWITCH2, J4 PGM_SWITCH3, J5 PGM_SWITCH2, J6 E1, J7 P7, J8 P7, J9 P10, Q1 3107B, Q10 3107B, Q2 3107B, Q3 kp103l, Q4 3107B, Q6 3107B, Q7 3107B, Q8 3107B, SW2 SW_Rotary12, SW3 SW_Rotary12

Commit message: w
Parts:
- added C17: x, Capacitor_THT:CP_Radial_D5.0mm_P2.50mm, F.Cu at (142.2, 78.2)
- added C18: x, Capacitor_THT:CP_Radial_D5.0mm_P2.50mm, F.Cu at (136.1, 74.7)
- added R39: 1k, Resistor_SMD:R_0603_1608Metric_Pad1.05x0.95mm_HandSolder, F.Cu at (142.2, 72.3)
- added R41: 100, Resistor_SMD:R_0603_1608Metric_Pad1.05x0.95mm_HandSolder, F.Cu at (147.5, 74.7)
- added R5: 47k, Resistor_SMD:R_0603_1608Metric_Pad1.05x0.95mm_HandSolder, F.Cu at (131.7, 62.0)
- added R51: 1k, Resistor_SMD:R_0603_1608Metric_Pad1.05x0.95mm_HandSolder, F.Cu at (147.5, 78.7)
- R1: value 5M11 -> 7k5; footprint Resistor_THT:R_Axial_DIN0617_L17.0mm_D6.0mm_P7.62mm_Vertical -> Resistor_THT:R_Axial_DIN0414_L11.9mm_D4.5mm_P5.08mm_Vertical
- R10, R35: value x -> 5k6
- R11: value x -> 3k
- R12: value 220k -> 51
- R13: value 220k -> 3k
- R15: value x -> 402
- R16: value x -> 390
- R17: value x -> 150
- R18, R21, R24, R27: value x -> 56k
- R19, R22, R25, R28, R30: value x -> 357
- R20, R23, R26, R29: value x -> 240
- R3: value 7k5 -> 21,8
- R31: value x -> 165
- R33, R37: value x -> 110
- R36: value x -> 10
- R38, R47: value x -> 1k
- R4: footprint Resistor_THT:R_Axial_DIN0516_L15.5mm_D5.0mm_P30.48mm_Horizontal -> Resistor_SMD:R_0603_1608Metric_Pad1.05x0.95mm_HandSolder
- R42, R45: value x -> 2k2
- R43: value x -> 15
- R44: value x -> 510
- R46: value x -> 680
- R48: value x -> 55,6
- R53, R54: value x -> 1M
- R55: renamed from R5; value x -> 2,49k
- R56: value x -> 2,49k
- RV57: renamed from RV1; value 220k -> 1k5
- moved R13 64.5 mm to (135.6, 117.9), turned to 180 degrees
- moved C7 38.9 mm to (138.2, 62.0)
- moved RV6 35.6 mm to (125.0, 57.9)
- moved C15 14.5 mm to (122.9, 68.1)
- moved C14 8.07 mm to (147.7, 68.1), turned to 180 degrees
- moved J8 7.27 mm to (126.0, 83.3)
- moved R32 6.02 mm to (131.6, 66.0)
- moved R33 6.00 mm to (131.6, 70.1)
- moved Q6 5.61 mm to (128.0, 77.2)
- moved R36 5.40 mm to (136.3, 78.7), turned to 180 degrees
- moved J10 4.32 mm to (144.8, 56.4)
- renumbered C17 to C21
Connections:
- RV6 pad 1: Net-(C7-Pad1) -> Net-(R5-Pad2)
